Commit message: small improvements

File: models/tiago_description/tiago.urdf (robot description, URDF)
Before this commit: robot tiago, 31 links, 30 joints
Links:
- link torso_fixed_link: geometry collision box size=0.25 0.25 0.1; collision box size=0.4 0.25 0.04
- link torso_lift_link: geometry collision mesh filename=meshes/torso/torso_lift_collision.dae scale=1 1 1; visual mesh filename=meshes/torso/torso_lift_with_arm.stl scale=1 1 1

Commit message: make gripper link heavier

File: models/tiago_description/tiago.urdf (robot description, URDF)
Before this commit: robot tiago, 31 links, 30 joints
Links:
- link gripper_left_finger_link: mass 0.00109980 -> 0.1
- link gripper_right_finger_link: mass 0.00109980 -> 0.1
Joints:
- joint arm_3_joint: limit lower=-3.53429173529 upper=1.8 effort=17.86 velocity=4.58 -> lower=-3.53429173529 upper=1.57079632679 effort=17.86 velocity=4.58
- joint arm_6_joint: limit lower=-1.41371669412 upper=1.8 effort=6.6 velocity=1.76 -> lower=-1.41371669412 upper=1.41371669412 effort=6.6 velocity=1.76
