Commit message: make gripper collision box wider

File: models/tiago_description/tiago.urdf (robot description, URDF)
Before this commit: robot tiago, 31 links, 30 joints
Links:
- link gripper_left_finger_link: geometry collision box size=0.01 0.1 0.11; visual mesh filename=meshes/gripper/gripper_finger_link.stl
- link gripper_right_finger_link: geometry collision box size=0.01 0.1 0.11; visual mesh filename=meshes/gripper/gripper_finger_link.stl scale=-1 -1 1
